Commit message: Initial commit (Modified controllers to Effort controllers)

File: robotiq_3f_gripper_visualization/cfg/robotiq-3f-gripper_articulated.urdf (robot description, URDF)
Before this commit: robot robotiq-3f-gripper_articulated, 13 links, 12 joints
Joints:
- joint finger_1_joint_1: limit lower=0 upper=3.1416 effort=100 velocity=100 -> lower=0 upper=3.1416 effort=${e1} velocity=${s1}
- joint finger_1_joint_2: limit lower=0 upper=3.1416 effort=100 velocity=100 -> lower=0 upper=3.1416 effort=${e1} velocity=${s1}
- joint finger_1_joint_3: limit lower=0 upper=3.1416 effort=100 velocity=100 -> lower=0 upper=3.1416 effort=${e1} velocity=${s1}
- joint finger_2_joint_1: limit lower=0 upper=3.1416 effort=100 velocity=100 -> lower=0 upper=3.1416 effort=${e1} velocity=${s1}
- joint finger_2_joint_2: limit lower=0 upper=3.1416 effort=100 velocity=100 -> lower=0 upper=3.1416 effort=${e1} velocity=${s1}
- joint finger_2_joint_3: limit lower=0 upper=3.1416 effort=100 velocity=100 -> lower=0 upper=3.1416 effort=${e1} velocity=${s1}
- joint finger_middle_joint_1: limit lower=0 upper=3.1416 effort=100 velocity=100 -> lower=0 upper=3.1416 effort=${e1} velocity=${s1}
- joint finger_middle_joint_2: limit lower=0 upper=3.1416 effort=100 velocity=100 -> lower=0 upper=3.1416 effort=${e1} velocity=${s1}
- joint finger_middle_joint_3: limit lower=0 upper=3.1416 effort=100 velocity=100 -> lower=0 upper=3.1416 effort=${e1} velocity=${s1}
- joint palm_finger_1_joint: limit lower=-0.16 upper=0.25 effort=100 velocity=100 -> lower=-0.16 upper=0.25 effort=${e1} velocity=${s1}
- joint palm_finger_2_joint: limit lower=-0.25 upper=0.16 effort=100 velocity=100 -> lower=-0.25 upper=0.16 effort=${e1} velocity=${s1}

File: robotiq_3f_gripper_visualization/cfg/robotiq-3f-gripper_articulated_macro_old.xacro (robot description, xacro)
@@ -6,8 +6,6 @@
 -->
 <robot xmlns:xacro="http://ros.org/wiki/xacro">
-        <xacro:property name="s1" value="0.85" />
-        <xacro:property name="e1" value="40" />
         <xacro:include filename="$(find robotiq_3f_gripper_visualization)/cfg/robotiq-3f-gripper_finger_articulated_macro.xacro" />
-        <xacro:macro name="robotiq-3f-gripper_articulated" params="prefix *origin reflect parent">
+        <xacro:macro name="robotiq-3f-gripper_articulated" params="prefix">
         <xacro:robotiq-3f-gripper_finger_articulated prefix="${prefix}finger_1_"/>
         <xacro:robotiq-3f-gripper_finger_articulated prefix="${prefix}finger_2_"/>
@@ -32,8 +30,4 @@
 			</collision>
 		</link>
-	    <gazebo reference="${prefix}palm">
-      		<mu1>1.1</mu1>
-      		<mu2>1.1</mu2>
-    	</gazebo>
         <inertial>
             <origin xyz="0 0 0" rpy="0 0 0"/>
@@ -48,5 +42,5 @@
 			<axis xyz="0 1 0"/>
 			<origin xyz="-0.0455 0.0214 0.036" rpy="0 3.1416 -1.57"/>
-                        <limit lower="-0.1784" upper="0.192" effort="100" velocity="${s1}"/>
+			<limit lower="-0.1784" upper="0.192" effort="100" velocity="100"/>
 		</joint>
 		<joint name="${prefix}palm_finger_2_joint" type="revolute">
@@ -55,5 +49,5 @@
 			<axis xyz="0 1 0"/>
 			<origin xyz="-0.0455 0.0214 -0.036" rpy="0 3.1416 -1.57"/>
-                        <limit lower="-0.192" upper="0.1784" effort="100" velocity="${s1}"/>
+			<limit lower="-0.192" upper="0.1784" effort="100" velocity="100"/>
 		</joint>
 		<joint name="${prefix}palm_finger_middle_joint" type="fixed">
@@ -63,27 +57,4 @@
 			<origin xyz="0.0455 0.0214 0" rpy="0 0 1.57"/>
 		</joint>
-		<joint name="${prefix}robotiq_hand_joint" type="fixed">
-      		<insert_block name="origin"/>
-      		<parent link="${parent}"/>
-      		<child link="${prefix}palm"/>
-    	</joint>
-    <transmission name="${prefix}palm_finger_1_trans">
-      <type>transmission_interface/SimpleTransmission</type>
-      <joint name="${prefix}palm_finger_1_joint">
-        <hardwareInterface>hardware_interface/EffortJointInterface</hardwareInterface>
-      </joint>
-      <actuator name="${prefix}palm_finger_1_motor">
-        <mechanicalReduction>1</mechanicalReduction>
-      </actuator>
-    </transmission>
-    <transmission name="${prefix}palm_finger_2_trans">
-      <type>transmission_interface/SimpleTransmission</type>
-      <joint name="${prefix}palm_finger_2_joint">
-        <hardwareInterface>hardware_interface/EffortJointInterface</hardwareInterface>
-      </joint>
-      <actuator name="${prefix}palm_finger_2_motor">
-        <mechanicalReduction>1</mechanicalReduction>
-      </actuator>
-    </transmission>
 		<!-- end of joint list -->
 	</xacro:macro>

File: robotiq_3f_gripper_visualization/cfg/robotiq-3f-gripper_finger_articulated_macro.xacro (robot description, xacro)
@@ -6,5 +6,8 @@
 -->
 <robot xmlns:xacro="http://ros.org/wiki/xacro">
+        <xacro:property name="s1" value="50.88" />
+        <xacro:property name="e1" value="100" />
         <xacro:macro name="robotiq-3f-gripper_finger_articulated" params="prefix">
+		<xacro:include filename="$(find robotiq_3f_gripper_visualization)/cfg/robotiq.transmission.xacro" />
 		<!-- link list -->
 		<link name="${prefix}link_0">
@@ -33,4 +36,8 @@
             </inertial>
 		</link>
+		<gazebo reference="${prefix}link_0">
+      		<mu1>1.1</mu1>
+      		<mu2>1.1</mu2>
+    	</gazebo>
 		<link name="${prefix}link_1">
 			<visual>
@@ -54,4 +61,8 @@
             </inertial>
 		</link>
+		<gazebo reference="${prefix}link_1">
+      		<mu1>1.1</mu1>
+      		<mu2>1.1</mu2>
+    	</gazebo>
 		<link name="${prefix}link_2">
 			<!--
@@ -80,4 +91,8 @@
             </inertial>
 		</link>
+		<gazebo reference="${prefix}link_2">
+      		<mu1>1.1</mu1>
+      		<mu2>1.1</mu2>
+    	</gazebo>
 		<link name="${prefix}link_3">
 			<visual>
@@ -101,6 +116,11 @@
             </inertial>
 		</link>
+		<gazebo reference="${prefix}link_3">
+      		<mu1>1.1</mu1>
+      		<mu2>1.1</mu2>
+    	</gazebo>
 		<!-- end of link list -->
 		<!-- joint list -->
+		<xacro:robotiq_transmission prefix="${prefix}" />
 		<joint name="${prefix}joint_1" type="revolute">
 			<parent link="${prefix}link_0"/>
@@ -108,5 +128,5 @@
 			<axis xyz="0 0 1"/>
 			<origin xyz="0.020 0 0" rpy="0 0 0"/>
-			<limit lower="0.0495" upper="1.2218" effort="100" velocity="100"/>
+                        <limit lower="0.0495" upper="1.2218" effort="${e1}" velocity="${s1}"/>
 		</joint>
 		<joint name="${prefix}joint_2" type="revolute">
@@ -115,5 +135,5 @@
 			<axis xyz="0 0 1"/>
 			<origin xyz="0.050 -.028 0" rpy="0 0 -0.52"/>
-			<limit lower="0.0" upper="1.5708" effort="100" velocity="100"/>
+                        <limit lower="0.0" upper="1.5708" effort="${e1}" velocity="${s1}"/>
 		</joint>
 		<joint name="${prefix}joint_3" type="revolute">
@@ -122,5 +142,5 @@
 			<axis xyz="0 0 1"/>
 			<origin xyz="0.039 0 0" rpy="0 0 0"/>
-			<limit lower="-1.2217" upper="-0.0523" effort="100" velocity="100"/>
+                        <limit lower="-1.2217" upper="-0.074532925" effort="${e1}" velocity="${s1}"/>
 		</joint>
 		<!-- end of joint list -->

File: robotiq_3f_gripper_visualization/cfg/robotiq_hand_macro.urdf.xacro (robot description, xacro)
@@ -6,5 +6,5 @@
 there are multiple hands then a prefix followed by an "_" is needed.
 -->
-<robot xmlns:xacro="http://www.ros.org/wiki/xacro" name="robotiq_hand">
+<robot xmlns:xacro="http://ros.org/wiki/xacro" name="robotiq_hand">
   <xacro:macro name="robotiq_finger" params="prefix">
     <!-- Link list -->
@@ -38,4 +38,5 @@
       <mu1>1.1</mu1>
       <mu2>1.1</mu2>
+      <selfCollide>true</selfCollide>
     </gazebo>
     <!-- Link 1 -->
@@ -71,4 +72,5 @@
       <mu1>1.1</mu1>
       <mu2>1.1</mu2>
+      <selfCollide>true</selfCollide>
     </gazebo>
     <!-- Link 2 -->
@@ -102,4 +104,5 @@
       <mu1>1.1</mu1>
       <mu2>1.1</mu2>
+      <selfCollide>true</selfCollide>
     </gazebo>
     <!-- Link 3 -->
@@ -133,4 +136,5 @@
       <mu1>1.1</mu1>
       <mu2>1.1</mu2>
+      <selfCollide>true</selfCollide>
     </gazebo>
     <!-- Link proximal actuating hinge -->
@@ -162,4 +166,5 @@
       <mu1>1.1</mu1>
       <mu2>1.1</mu2>
+      <selfCollide>true</selfCollide>
     </gazebo>
     <!-- Link paraproximal actuating hinge -->
@@ -192,4 +197,5 @@
       <mu1>1.1</mu1>
       <mu2>1.1</mu2>
+      <selfCollide>true</selfCollide>
     </gazebo>
     <!-- Link proximal actuating bar -->
@@ -221,4 +227,5 @@
       <mu1>1.1</mu1>
       <mu2>1.1</mu2>
+      <selfCollide>true</selfCollide>
     </gazebo>
     <!-- Link paraproximal bar -->
@@ -250,4 +257,5 @@
       <mu1>1.1</mu1>
       <mu2>1.1</mu2>
+      <selfCollide>true</selfCollide>
     </gazebo>
     <!-- Link median actuating hinge -->
@@ -279,4 +287,5 @@
       <mu1>1.1</mu1>
       <mu2>1.1</mu2>
+      <selfCollide>true</selfCollide>
     </gazebo>
     <!-- Link median bar -->
@@ -308,4 +317,5 @@
       <mu1>1.1</mu1>
       <mu2>1.1</mu2>
+      <selfCollide>true</selfCollide>
     </gazebo>
     <!-- Link paramedian hinge -->
@@ -337,4 +347,5 @@
       <mu1>1.1</mu1>
       <mu2>1.1</mu2>
+      <selfCollide>true</selfCollide>
     </gazebo>
     <!-- Link median bar underactuated -->
@@ -366,4 +377,5 @@
       <mu1>1.1</mu1>
       <mu2>1.1</mu2>
+      <selfCollide>true</selfCollide>
     </gazebo>
     <!-- Link paradistal hinge -->
@@ -395,4 +407,5 @@
       <mu1>1.1</mu1>
       <mu2>1.1</mu2>
+      <selfCollide>true</selfCollide>
     </gazebo>
     <!-- End of link list -->
